File: homee_kicad.kicad_sch (KiCad schematic)
At the start: 28 parts, among them J1 Screw_Terminal_01x02, J2 USB_B_Micro, J3 Screw_Terminal_01x02, K1 SANYOU_SRD_Form_C, Q2 Q_NPN_Darlington_CBE, T1 Transformer_1P_1S, U1 ESP-01v090, U2 LD1117S33TR_SOT223, U4 PC817

Commit message: hello
Parts:
- T1: footprint PC-24-1000:XFMR_PC-24-1000 -> WE-PPTI_1006:WE-PPTI_1006_L10.2W6.73H4.19
Changed lines of the file:
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@@
 			)
 		)
-		(property "Footprint" "PC-24-1000:XFMR_PC-24-1000"
+		(property "Footprint" "WE-PPTI_1006:WE-PPTI_1006_L10.2W6.73H4.19"
 			(at 91.44 168.91 0)
 			(effects
