File: homee_kicad.kicad_sch (KiCad schematic)
At the start: 20 parts, among them K2 SANYOU_SRD_Form_C, Q1 Q_NPN_Darlington_CBE, T1 Transformer_1P_1S, U1 ESP-01v090, U2 LD1117S33TR_SOT223, U3 PC817

Commit message: Relay Circuit Usb Circuit Pull up Circuit
Parts:
- added C3: C, Capacitor_SMD:CP_Elec_3x5.3, symbol Device:C
- added D7: D, Diode_SMD:D_0201_0603Metric, symbol Device:D
- added D8: LED, Diode_SMD:D_0201_0603Metric, symbol Device:LED
- added D9: D, symbol Device:D
- added J2: USB_B_Micro, Connector_USB:USB_Micro-AB_Molex_47590-0001, symbol Connector:USB_B_Micro
- added K1: SANYOU_SRD_Form_C, Relay_THT:Relay_SPDT_SANYOU_SRD_Series_Form_C, symbol Relay:SANYOU_SRD_Form_C
- added Q2: Q_NPN_Darlington_CBE, Package_TO_SOT_THT:TO-92_Horizontal1, symbol Device:Q_NPN_Darlington_CBE
- added R10: 10k, Resistor_SMD:R_1020_2550Metric, symbol Device:R
- added R7, R8, R9: R, Resistor_SMD:R_1020_2550Metric, symbol Device:R
- added U4: PC817, Package_DIP:DIP-4_W7.62mm, symbol Isolator:PC817
- R4, R5, R6: value R -> 10k
Connections:
- net Earth: now also Q2.1 (C), R8.1, R8.2
- net GND: now also J2.5 (GND)
- net GPIO0: now also R4.2, U4.2; no longer U3.2
- net VCC: now also R4.1, R5.1, R6.1, D9.1 (K), R10.1
- net RST: now reaches U1.5 (RST)
- net RST: now also R6.2, C3.1; no longer R6.1
- net TX: now reaches U1.1 (UTXD)
- net TX: now also J2.2 (D-)
- net CH_PD: now reaches U1.3 (CH_PD)
- net GPIO2: now reaches U1.4 (GPIO2)
- net GPIO2: now also U3.2, R10.2
- net RX: now reaches U1.8 (URXD)
- net RX: now also J2.3 (D+)
- new net: R7.2, U4.1
- new net: Q2.2 (B), U4.3
- new net: R7.1, U4.4
- new net: D9.2 (A), J2.1 (VBUS)
- new net: D7.2 (A), D8.1 (K), K1.2, Q2.3 (E)
- new net: D7.1 (K), K1.5, R9.2
- new net: D8.2 (A), R9.1
- no-connect marks 8 -> 9
Other:
- note added: "MICRO USB CIRCUIT"
- note added: "PULL UP CIRCUIT"
- note added: "RELAY 1 CIRCUIT"
- note added: "RELAY 2 CIRCUIT"
- note removed: "RELAY CIRCUIT"
- moved on the sheet: R4, R5, R6, U1

Commit message: oe
Parts:
- added D10: LED, Diode_SMD:D_0201_0603Metric_Pad0.64x0.40mm_HandSolder, symbol Device:LED
- added R11: R, Capacitor_THT:CP_Radial_Tantal_D4.5mm_P2.50mm, symbol Device:R
- D9: footprint (none) -> Diode_SMD:D_0201_0603Metric
- J2: footprint Connector_USB:USB_Micro-AB_Molex_47590-0001 -> Connector_USB:USB_Micro-B_Amphenol_10103594-0001LF_Horizontal
Connections:
- net GND: now also D10.1 (K)
- net TX: now also R11.2; no longer J2.2 (D-)
- new net: D10.2 (A), R11.1
- no-connect marks 9 -> 10
Changed lines of the file:
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@@
 	)
 	(no_connect
+		(at 34.29 175.26)
+	)
+	(no_connect
 		(at 201.93 100.33)
 	)
@@
 	(wire
 		(pts
-			(xy 34.29 175.26) (xy 40.64 175.26)
+			(xy 54.61 101.6) (xy 66.04 101.6)
 		)
 		(stroke
@@
 	(wire
 		(pts
-			(xy 54.61 101.6) (xy 66.04 101.6)
+			(xy 195.58 36.83) (xy 195.58 41.91)
 		)
 		(stroke
@@
 	(wire
 		(pts
-			(xy 195.58 36.83) (xy 195.58 41.91)
+			(xy 245.11 147.32) (xy 245.11 151.13)
 		)
 		(stroke
@@
 	(wire
 		(pts
-			(xy 245.11 147.32) (xy 245.11 151.13)
+			(xy 245.11 100.33) (xy 256.54 100.33)
 		)
 		(stroke
@@
 	(wire
 		(pts
-			(xy 245.11 100.33) (xy 256.54 100.33)
+			(xy 93.98 167.64) (xy 93.98 168.91)
 		)
 		(stroke
@@
 	(wire
 		(pts
-			(xy 93.98 167.64) (xy 93.98 168.91)
+			(xy 149.86 160.02) (xy 149.86 165.1)
 		)
 		(stroke
@@
 	(wire
 		(pts
-			(xy 149.86 160.02) (xy 149.86 165.1)
+			(xy 86.36 170.18) (xy 101.6 170.18)
 		)
 		(stroke
@@
 	(wire
 		(pts
-			(xy 86.36 170.18) (xy 101.6 170.18)
+			(xy 127 78.74) (xy 127 93.98)
 		)
 		(stroke
@@
 	(wire
 		(pts
+			(xy 54.61 78.74) (xy 127 78.74)
+		)
+		(stroke
+			(width 0)
+			(type default)
+		)
+	)
+	(wire
+		(pts
 			(xy 195.58 41.91) (xy 200.66 41.91)
 		)
@@
 		)
 	)
-	(label "TX"
-		(at 38.1 175.26 0)
-		(fields_autoplaced yes)
-		(effects
-			(font
-				(size 1.27 1.27)
-			)
-			(justify left bottom)
-		)
-	)
 	(label "GND"
 		(at 118.11 93.98 0)
@@
 			)
 		)
-		(property "Footprint" ""
+		(property "Footprint" "Diode_SMD:D_0201_0603Metric"
 			(at 38.1 167.64 0)
 			(effects
@@
 			)
 		)
-		(property "Footprint" "Connector_USB:USB_Micro-AB_Molex_47590-0001"
+		(property "Footprint" "Connector_USB:USB_Micro-B_Amphenol_10103594-0001LF_Horizontal"
 			(at 30.48 173.99 0)
 			(effects
@@
 	)
 	(symbol
+		(lib_id "Device:R")
+		(at 54.61 90.17 0)
+		(unit 1)
+		(exclude_from_sim no)
+		(in_bom yes)
+		(on_board yes)
+		(dnp no)
+		(fields_autoplaced yes)
+		(property "Reference" "R11"
+			(at 57.15 88.8999 0)
+			(effects
+				(font
+					(size 1.27 1.27)
+				)
+				(justify left)
+			)
+		)
+		(property "Value" "R"
+			(at 57.15 91.4399 0)
+			(effects
+				(font
+					(size 1.27 1.27)
+				)
+				(justify left)
+			)
+		)
+		(property "Footprint" "Capacitor_THT:CP_Radial_Tantal_D4.5mm_P2.50mm"
+			(at 52.832 90.17 90)
+			(effects
+				(font
+					(size 1.27 1.27)
+				)
+				(hide yes)
+			)
+		)
+		(property "Datasheet" "~"
+			(at 54.61 90.17 0)
+			(effects
+				(font
+					(size 1.27 1.27)
+				)
+				(hide yes)
+			)
+		)
+		(property "Description" "Resistor"
+			(at 54.61 90.17 0)
+			(effects
+				(font
+					(size 1.27 1.27)
+				)
+				(hide yes)
+			)
+		)
+		(pin "2"
+		)
+		(pin "1"
+		)
+		(instances
+			(project ""
+				(path "/b4bceb5a-cab3-4f49-a303-5f79905a3ea8"
+					(reference "R11")
+					(unit 1)
+				)
+			)
+		)
+	)
+	(symbol
 		(lib_id "Relay:SANYOU_SRD_Form_C")
 		(at 209.55 92.71 180)
@@
 					(unit 1)
 				)
+			)
+		)
+	)
+	(symbol
+		(lib_id "Device:LED")
+		(at 54.61 82.55 270)
+		(unit 1)
+		(exclude_from_sim no)
+		(in_bom yes)
+		(on_board yes)
+		(dnp no)
+		(fields_autoplaced yes)
+		(property "Reference" "D10"
+			(at 57.15 79.6924 90)
+			(effects
+				(font
+					(size 1.27 1.27)
+				)
+				(justify left)
+			)
+		)
+		(property "Value" "LED"
+			(at 57.15 82.2324 90)
+			(effects
+				(font
+					(size 1.27 1.27)
+				)
+				(justify left)
+			)
+		)
+		(property "Footprint" "Diode_SMD:D_0201_0603Metric_Pad0.64x0.40mm_HandSolder"
+			(at 54.61 82.55 0)
+			(effects
+				(font
+					(size 1.27 1.27)
+				)
+				(hide yes)
+			)
+		)
+		(property "Datasheet" "~"
+			(at 54.61 82.55 0)
+			(effects
+				(font
+					(size 1.27 1.27)
+				)
+				(hide yes)
+			)
+		)
+		(property "Description" "Light emitting diode"
+			(at 54.61 82.55 0)
+			(effects
+				(font
+					(size 1.27 1.27)
+				)
+				(hide yes)
+			)
+		)
+		(pin "1"
+		)
+		(pin "2"
+		)
+		(instances
+			(project ""
+				(path "/b4bceb5a-cab3-4f49-a303-5f79905a3ea8"
+					(reference "D10")
+					(unit 1)
+				)
