File: homee_kicad.kicad_pcb (KiCad board)
At the start: 2 copper layers, 51.9 x 47 mm, 21 parts, among them J1 Screw_Terminal_01x04, J2 476421001, K2 SANYOU_SRD_Form_C, Q1 2N7002, U1 ESP-01v090, U2 LD1117S33TR_SOT223, U4 PC817

Commit message: je croyais que j'avais fini :(
Parts:
- moved D7 11.4 mm to (130.6, 112.4), turned to 90 degrees
- moved U2 2.50 mm to (124.1, 114.8)
- moved C2 2.15 mm to (117.3, 113.5)
- moved R1 2.10 mm to (116.2, 108.8), turned to -90 degrees
- moved R9 1.71 mm to (132.1, 107.9)
- moved D8 1.51 mm to (124.3, 108.0)
- moved D1 1.48 mm to (121.8, 108.0)
- moved C1 1.44 mm to (117.3, 116.8)
Routing:
- net Net-(D7-A): track 58.4 -> 41.6 mm
- net GND: track 88.1 -> 97.1 mm
- net +5V: track 47.8 -> 41.8 mm, vias 1 -> 0
Other:
- board size 51.9 x 47 mm -> 52.2 x 44.8 mm
