File: homee_kicad.kicad_pcb (KiCad board)
At the start: 2 copper layers, 56.1 x 45 mm, 21 parts, among them J1 Screw_Terminal_01x04, J2 476421001, K2 SANYOU_SRD_Form_C, Q1 2N7002, U1 ESP-01v090, U2 LD1117S33TR_SOT223, U4 PC817

Commit message: PLZ BE THE LAST TIME :'(
Parts:
- D7, R1, R5, R6, R9: moved to B.Cu
- J1: footprint TerminalBlock_Phoenix:TerminalBlock_Phoenix_PT-1,5-4-3.5-H_1x04_P3.50mm_Horizontal -> TerminalBlock:TerminalBlock_Xinya_XY308-2.54-4P_1x04_P2.54mm_Horizontal
- moved U2 71.0 mm to (118.0, 68.0), turned to 180 degrees
- moved C2 69.9 mm to (111.8, 69.2), turned to 90 degrees
- moved C1 67.3 mm to (124.2, 69.2), turned to 90 degrees
- moved R4 60.3 mm to (102.4, 70.8), turned to 180 degrees
- moved D1 56.2 mm to (101.8, 64.6), turned to 0 degrees
- moved R9 56.0 mm to (107.4, 65.0)
- moved D8 53.9 mm to (112.1, 64.5), turned to 180 degrees
- moved BC1 50.3 mm to (128.0, 80.6)
- moved J2 50.1 mm to (108.1, 96.8)
- moved R5 50.0 mm to (107.2, 69.9)
- moved D7 49.5 mm to (115.5, 68.0), turned to 90 degrees
- moved K2 49.0 mm to (119.9, 73.6)
- moved J1 48.9 mm to (118.0, 96.0)
- moved U4 47.5 mm to (106.4, 81.3), turned to 0 degrees
- moved C3 47.2 mm to (102.5, 69.4)
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Routing:
- net VCC: track 0.00 -> 55.6 mm, vias 0 -> 1
- net /L IN: track 0.00 -> 42.7 mm
- net Net-(D7-A): track 0.00 -> 39.3 mm
- net GND: track 0.00 -> 23.5 mm, vias 0 -> 1
- net /RX: track 0.00 -> 20.0 mm, vias 0 -> 1
- net +5V: track 0.00 -> 18.3 mm, vias 0 -> 1
- net /GPIO0: track 0.11 -> 12.1 mm, vias 0 -> 1
- net /NO: track 0.00 -> 9.93 mm
- net Net-(D1-A): track 0.00 -> 9.48 mm
- net /NC: track 0.00 -> 9.31 mm
- net Net-(R7-Pad2): track 0.00 -> 8.62 mm
- net /RST: track 0.00 -> 7.02 mm
- net /RELAY: track 0.11 -> 5.21 mm
- net /TX: track 0.00 -> 3.57 mm
- net /N IN: track 0.00 -> 3.37 mm
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Other:
- board size 56.1 x 45 mm -> 50 x 38 mm
