File: _autosave-homee_kicad.kicad_pcb (KiCad board)
At the start: 2 copper layers, 56.1 x 45 mm, 21 parts, among them J1 Screw_Terminal_01x04, J2 476421001, K2 SANYOU_SRD_Form_C, Q1 2N7002, U1 ESP-01v090, U2 LD1117S33TR_SOT223, U4 PC817

Commit message: oeoe
Parts:
- moved Q1 22.3 mm to (105.1, 139.4)
- moved D7 22.3 mm to (110.0, 139.4)
- moved C2 19.0 mm to (96.1, 131.8)
- moved C1 19.0 mm to (96.1, 128.4)
- moved U2 19.0 mm to (89.8, 131.0)
- moved U4 3.45 mm to (108.8, 132.1)
- moved R4 3.45 mm to (115.0, 133.1)
- moved R7 3.45 mm to (114.1, 136.2)
- moved R8 3.45 mm to (108.4, 136.1)
- moved U1 3.45 mm to (105.7, 124.9)
Routing:
- net (no net): vias 1 -> 2
Changed lines of the file:
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@@
 	(footprint "Capacitor_SMD:C_1210_3225Metric"
 		(layer "F.Cu")
-		(at 113.7 139.05 180)
+		(at 96.075 131.825 180)
 		(descr "Capacitor SMD 1210 (3225 Metric), square (rectangular) end terminal, IPC_7351 nominal, (Body size source: IPC-SM-782 page 76, https://www.pcb-3d.com/wordpress/wp-content/uploads/ipc-sm-782a_amendment_1_and_2.pdf), generated with kicad-footprint-generator")
 		(tags "capacitor")
@@
 	(footprint "Package_TO_SOT_SMD:SOT-23"
 		(layer "F.Cu")
-		(at 108.6125 117.325)
+		(at 105.1375 139.4)
 		(descr "SOT, 3 Pin (https://www.jedec.org/system/files/docs/to-236h.pdf variant AB), generated with kicad-footprint-generator ipc_gullwing_generator.py")
 		(tags "SOT TO_SOT_SMD")
@@
 	(footprint "Package_TO_SOT_SMD:SOT-223-3_TabPin2"
 		(layer "F.Cu")
-		(at 107.475 138.225 90)
+		(at 89.85 131 90)
 		(descr "module CMS SOT223 4 pins")
 		(tags "CMS SOT")
@@
 	(footprint "Package_DIP:SMDIP-4_W7.62mm"
 		(layer "F.Cu")
-		(at 109.025 128.7 180)
+		(at 108.775 132.145 180)
 		(descr "4-lead surface-mounted (SMD) DIP package, row spacing 7.62 mm (300 mils)")
 		(tags "SMD DIP DIL PDIP SMDIP 2.54mm 7.62mm 300mil")
@@
 	(footprint "Resistor_SMD:R_0805_2012Metric_Pad1.20x1.40mm_HandSolder"
 		(layer "F.Cu")
-		(at 115.275 129.65 90)
+		(at 115.025 133.095 90)
 		(descr "Resistor SMD 0805 (2012 Metric), square (rectangular) end terminal, IPC_7351 nominal with elongated pad for handsoldering. (Body size source: IPC-SM-782 page 72, https://www.pcb-3d.com/wordpress/wp-content/uploads/ipc-sm-782a_amendment_1_and_2.pdf), generated with kicad-footprint-generator")
 		(tags "resistor handsolder")
@@
 	(footprint "Capacitor_SMD:C_1210_3225Metric"
 		(layer "F.Cu")
-		(at 113.68 135.635 180)
+		(at 96.055 128.41 180)
 		(descr "Capacitor SMD 1210 (3225 Metric), square (rectangular) end terminal, IPC_7351 nominal, (Body size source: IPC-SM-782 page 76, https://www.pcb-3d.com/wordpress/wp-content/uploads/ipc-sm-782a_amendment_1_and_2.pdf), generated with kicad-footprint-generator")
 		(tags "capacitor")
@@
 	(footprint "Resistor_SMD:R_0805_2012Metric_Pad1.20x1.40mm_HandSolder"
 		(layer "F.Cu")
-		(at 114.325 132.725 180)
+		(at 114.075 136.17 180)
 		(descr "Resistor SMD 0805 (2012 Metric), square (rectangular) end terminal, IPC_7351 nominal with elongated pad for handsoldering. (Body size source: IPC-SM-782 page 72, https://www.pcb-3d.com/wordpress/wp-content/uploads/ipc-sm-782a_amendment_1_and_2.pdf), generated with kicad-footprint-generator")
 		(tags "resistor handsolder")
@@
 	(footprint "Diode_SMD:D_1210_3225Metric_Pad1.42x2.65mm_HandSolder"
 		(layer "F.Cu")
-		(at 113.4375 117.375 180)
+		(at 109.975 139.45 180)
 		(descr "Diode SMD 1210 (3225 Metric), square (rectangular) end terminal, IPC_7351 nominal, (Body size source: http://www.tortai-tech.com/upload/download/2011102023233369053.pdf), generated with kicad-footprint-generator")
 		(tags "diode handsolder")
@@
 	(footprint "Resistor_SMD:R_0805_2012Metric_Pad1.20x1.40mm_HandSolder"
 		(layer "F.Cu")
-		(at 108.625 132.65 180)
+		(at 108.375 136.095 180)
 		(descr "Resistor SMD 0805 (2012 Metric), square (rectangular) end terminal, IPC_7351 nominal with elongated pad for handsoldering. (Body size source: IPC-SM-782 page 72, https://www.pcb-3d.com/wordpress/wp-content/uploads/ipc-sm-782a_amendment_1_and_2.pdf), generated with kicad-footprint-generator")
 		(tags "resistor handsolder")
@@
 	(footprint "Connector_PinSocket_2.54mm:PinSocket_2x04_P2.54mm_Vertical"
 		(layer "F.Cu")
-		(at 105.92 121.48 90)
+		(at 105.67 124.925 90)
 		(descr "Through hole straight socket strip, 2x04, 2.54mm pitch, double cols (from Kicad 4.0.7), script generated")
 		(tags "Through hole socket strip THT 2x04 2.54mm double row")
@@
 	)
 	(via
-		(at 115.325 126.8)
+		(at 111.2 136.095)
+		(size 1.6)
+		(drill 1.4)
+		(layers "F.Cu" "B.Cu")
+		(net 0)
+	)
+	(via
+		(at 115.075 130.245)
 		(size 1.6)
 		(drill 1.6)
@@
 	)
 	(segment
-		(start 105.39 127.43)
-		(end 105.5 127.43)
+		(start 105.14 130.875)
+		(end 105.25 130.875)
 		(width 0.6)
 		(layer "F.Cu")
@@
 	)
 	(segment
-		(start 113.01 127.43)
-		(end 112.9 127.43)
+		(start 112.76 130.875)
+		(end 112.65 130.875)
 		(width 0.6)
 		(layer "F.Cu")
